File: Hardware/flight_comp.kicad_sch (KiCad schematic)
At the start: 29 parts, among them J2 ARM_SWD_TC2030, J4 USB_C_Receptacle_USB2.0_16P, U1 STM32F405RGTx, U4 W25Q32JVSS, U5 24LC64, U8 USBLC6-2SC6, Y1 8mHz, Y2 32.768 kHz

Commit message: Minor changes in sensors and peripherals
Parts:
- added D4: WS2812B, LED_SMD:LED_WS2812B_PLCC4_5.0x5.0mm_P3.2mm, symbol LED:WS2812B
- added R21: 10k, symbol Device:R
- added R28, R29: R, symbol Device:R
- added R32: 0R, symbol Device:R
Connections:
- net +3.3V: now also R28.1, R29.1, R32.2
- net +3.3VB: now also R32.1
- net EEP_SCL: now also R29.2
- net EEP_SDA: now also R28.2
- net GND: now also D4.3 (VSS), R21.2
- net LED: now also U1.56 (PB4), D4.4 (DIN), R21.1; no longer U1.2 (PC13)
- net BAT_VSENCE: now reaches U1.20 (PA4)
- new net +5V: D4.1 (VDD)
- no-connect marks 9 -> 8
Other:
- moved on the sheet: C10, C11, C30, C31, C32, C33, J2, R7, U4, U5
