File: Hardware/flight_comp.kicad_sch (KiCad schematic)
At the start: 43 parts, among them J2 TC2030, J4 USB_C_Receptacle_USB2.0_16P, Q5 PMBT2222A, SW1 NRST, SW2 BOOT0, U1 STM32F405RGTx, U4 W25Q32JVSS, U5 24LC64, U8 USBLC6-2SC6, Y1 8mHz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

Commit message: GPS antenna connections, pps is connected to the mcu, pps diode replaced
Parts:
- removed Q5: PMBT2222A, Package_TO_SOT_SMD:SOT-23, symbol Transistor_BJT:PMBT2222A
Connections:
- net PPS: now reaches U1.9 (PC1)
- net at R33.2: now also BZ1.2 (-)
- no-connect marks 7 -> 6
Other:
- moved on the sheet: BZ1, R33
Changed lines of the file:
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@@
 		(at 148.59 86.36)
 	)
-	(no_connect
-		(at 148.59 55.88)
-	)
 	(wire
 		(pts
@@
 	(wire
 		(pts
-			(xy 248.92 25.4) (xy 248.92 26.67)
+			(xy 250.19 29.21) (xy 250.19 30.48)
 		)
 		(stroke
@@
 		)
 	)
+	(wire
+		(pts
+			(xy 245.11 35.56) (xy 250.19 35.56)
+		)
+		(stroke
+			(width 0)
+			(type default)
+		)
+	)
 	(global_label "TIM5_CH4"
 		(shape input)
@@
 	(global_label "BUZZ"
 		(shape input)
-		(at 233.68 36.83 180)
+		(at 237.49 35.56 180)
 		(fields_autoplaced yes)
 		(effects
@@
 		)
 		(property "Intersheetrefs" "${INTERSHEET_REFS}"
-			(at 225.6753 36.83 0)
+			(at 229.4853 35.56 0)
 			(effects
 				(font
@@
 		)
 	)
+	(global_label "PPS"
+		(shape input)
+		(at 148.59 55.88 180)
+		(fields_autoplaced yes)
+		(effects
+			(font
+				(size 1.27 1.27)
+			)
+			(justify right)
+		)
+		(property "Intersheetrefs" "${INTERSHEET_REFS}"
+			(at 141.8553 55.88 0)
+			(effects
+				(font
+					(size 1.27 1.27)
+				)
+				(justify right)
+				(hide yes)
+			)
+		)
+	)
 	(global_label "IMU_INT1"
 		(shape input)
@@
 	(symbol
 		(lib_id "power:GND")
-		(at 248.92 41.91 0)
-		(unit 1)
-		(exclude_from_sim no)
-		(in_bom yes)
-		(on_board yes)
-		(dnp no)
-		(fields_autoplaced yes)
-		(property "Reference" "#PWR0134"
-			(at 248.92 48.26 0)
-			(effects
-				(font
-					(size 1.27 1.27)
-				)
-				(hide yes)
-			)
-		)
-		(property "Value" "GND"
-			(at 248.92 46.99 0)
-			(effects
-				(font
-					(size 1.27 1.27)
-				)
-			)
-		)
-		(property "Footprint" ""
-			(at 248.92 41.91 0)
-			(effects
-				(font
-					(size 1.27 1.27)
-				)
-				(hide yes)
-			)
-		)
-		(property "Datasheet" ""
-			(at 248.92 41.91 0)
-			(effects
-				(font
-					(size 1.27 1.27)
-				)
-				(hide yes)
-			)
-		)
-		(property "Description" "Power symbol creates a global label with name \"GND\" , ground"
-			(at 248.92 41.91 0)
-			(effects
-				(font
-					(size 1.27 1.27)
-				)
-				(hide yes)
-			)
-		)
-		(pin "1"
-		)
-		(instances
-			(project "flight_comp"
-				(path "/99100214-bcab-4638-96e7-2342f837a8e5"
-					(reference "#PWR0134")
-					(unit 1)
-				)
-			)
-		)
-	)
-	(symbol
-		(lib_id "power:GND")
 		(at 130.81 43.18 0)
 		(unit 1)
@@
 	(symbol
 		(lib_id "power:+3.3V")
-		(at 248.92 25.4 0)
+		(at 250.19 29.21 0)
 		(unit 1)
 		(exclude_from_sim no)
@@
 		(fields_autoplaced yes)
 		(property "Reference" "#PWR0135"
-			(at 248.92 29.21 0)
+			(at 250.19 33.02 0)
 			(effects
 				(font
@@
 		)
 		(property "Value" "+3.3V"
-			(at 248.92 20.32 0)
+			(at 250.19 24.13 0)
 			(effects
 				(font
@@
 		)
 		(property "Footprint" ""
-			(at 248.92 25.4 0)
+			(at 250.19 29.21 0)
 			(effects
 				(font
@@
 		)
 		(property "Datasheet" ""
-			(at 248.92 25.4 0)
+			(at 250.19 29.21 0)
 			(effects
 				(font
@@
 		)
 		(property "Description" "Power symbol creates a global label with name \"+3.3V\""
-			(at 248.92 25.4 0)
+			(at 250.19 29.21 0)
 			(effects
 				(font
@@
 	)
 	(symbol
-		(lib_id "Transistor_BJT:PMBT2222A")
-		(at 246.38 36.83 0)
-		(unit 1)
-		(exclude_from_sim no)
-		(in_bom yes)
-		(on_board yes)
-		(dnp no)
-		(fields_autoplaced yes)
-		(property "Reference" "Q5"
-			(at 251.46 35.5599 0)
-			(effects
-				(font
-					(size 1.27 1.27)
-				)
-				(justify left)
-			)
-		)
-		(property "Value" "PMBT2222A"
-			(at 251.46 38.0999 0)
-			(effects
-				(font
-					(size 1.27 1.27)
-				)
-				(justify left)
-			)
-		)
-		(property "Footprint" "Package_TO_SOT_SMD:SOT-23"
-			(at 251.46 38.735 0)
-			(effects
-				(font
-					(size 1.27 1.27)
-					(italic yes)
-				)
-				(justify left)
-				(hide yes)
-			)
-		)
-		(property "Datasheet" "https://assets.nexperia.com/documents/data-sheet/PMBT2222A.pdf"
-			(at 246.38 36.83 0)
-			(effects
-				(font
-					(size 1.27 1.27)
-				)
-				(justify left)
-				(hide yes)
-			)
-		)
-		(property "Description" "600mA Ic, 40V Vce, NPN Transistor, SOT-23"
-			(at 246.38 36.83 0)
-			(effects
-				(font
-					(size 1.27 1.27)
-				)
-				(hide yes)
-			)
-		)
-		(pin "3"
-		)
-		(pin "2"
-		)
-		(pin "1"
-		)
-		(instances
-			(project ""
-				(path "/99100214-bcab-4638-96e7-2342f837a8e5"
-					(reference "Q5")
-					(unit 1)
-				)
-			)
-		)
-	)
-	(symbol
 		(lib_id "power:GND")
 		(at 128.27 106.68 0)
@@
 	(symbol
 		(lib_id "Device:R")
-		(at 237.49 36.83 90)
+		(at 241.3 35.56 90)
 		(unit 1)
 		(exclude_from_sim no)
@@
 		(fields_autoplaced yes)
 		(property "Reference" "R33"
-			(at 237.49 30.48 90)
+			(at 241.3 29.21 90)
 			(effects
 				(font
@@
 		)
 		(property "Value" "1k"
-			(at 237.49 33.02 90)
+			(at 241.3 31.75 90)
 			(effects
 				(font
@@
 		)
 		(property "Footprint" "Resistor_SMD:R_0603_1608Metric"
-			(at 237.49 38.608 90)
+			(at 241.3 37.338 90)
 			(effects
 				(font
@@
 		)
 		(property "Datasheet" "~"
-			(at 237.49 36.83 0)
+			(at 241.3 35.56 0)
 			(effects
 				(font
@@
 		)
 		(property "Description" "Resistor"
-			(at 237.49 36.83 0)
+			(at 241.3 35.56 0)
 			(effects
 				(font
@@
 	(symbol
 		(lib_id "Device:Buzzer")
-		(at 251.46 29.21 0)
+		(at 252.73 33.02 0)
 		(unit 1)
 		(exclude_from_sim no)
@@
 		(fields_autoplaced yes)
 		(property "Reference" "BZ1"
-			(at 255.27 27.9399 0)
+			(at 256.54 31.7499 0)
 			(effects
 				(font
@@
 		)
 		(property "Value" "Buzzer"
-			(at 255.27 30.4799 0)
+			(at 256.54 34.2899 0)
 			(effects
 				(font
@@
 		)
 		(property "Footprint" "Buzzer_Beeper:Buzzer_CUI_CPT-9019S-SMT"
-			(at 250.825 26.67 90)
+			(at 252.095 30.48 90)
 			(effects
 				(font
@@
 		)
 		(property "Datasheet" "~"
-			(at 250.825 26.67 90)
+			(at 252.095 30.48 90)
 			(effects
 				(font
@@
 		)
 		(property "Description" "Buzzer, polarized"
-			(at 251.46 29.21 0)
+			(at 252.73 33.02 0)
 			(effects
 				(font
