File: Hardware/sensors.kicad_sch (KiCad schematic)
At the start: 26 parts, among them IC1 BMP388, J1 Conn_Coaxial, J12 Conn_Coaxial, U13 LSM6DSO, U2 MAX-M10S, U3 74LVC1GU04

Commit message: Minor changes in sensors and peripherals
Parts:
- removed JP2: SolderJumper_3_Open, Jumper:SolderJumper-3_P1.3mm_Open_Pad1.0x1.5mm, symbol Jumper:SolderJumper_3_Open
- added R24, R25, R26, R27: R, symbol Device:R
Connections:
- net +3.3V: now also IC1.5 (SDO), R24.1, R25.1, R26.1, R27.1
- net BMP_SCL: now also R25.2
- net BMP_SDA: now also R24.2
- net GPS_SCL: now also R27.2
- net GPS_SDA: now also R26.2
- net IMU_INT1: now reaches U13.4 (INT1)
- no-connect marks 11 -> 10
Other:
- moved on the sheet: U3
