File: Hardware/flight_comp.kicad_pcb (KiCad board)
At the start: 2 copper layers, 86.8 x 49.2 mm, 116 parts, among them IC1 BMP388, J1 Conn_Coaxial, J12 Conn_Coaxial, J2 ARM_SWD_TC2030, J3 XT30, J4 USB_C_Receptacle_USB2.0_16P, J5 Conn_01x02, J6 Conn_01x02, J7 SERVO_CONN_01, J8 SERVO_CONN_02, J9 SERVO_CONN_02, Q1 FDN340P, Q2 DMP3013SFV, Q3 CSD17577Q3A, Q4 CSD17577Q3A, Q5 PMBT2222A, SW1 NRST, SW2 BOOT0, U1 STM32F405RGTx, U10 LTC4412, U11 UCC27517A, U12 UCC27517A, U13 LSM6DSO, U2 MAX-M10S, U3 74LVC1GU04, U4 W25Q32JVSS, U5 24LC64, U6 MP2331, U7 KA78M05, U8 USBLC6-2SC6, U9 LTC4412, Y1 8mHz, Y2 32.768 kHz

Commit message: 5V removed, PCB routing
Parts:
- removed C18: 0.33uF, Capacitor_SMD:C_0603_1608Metric
- removed C19, C24: 0.1uF, Capacitor_SMD:C_0603_1608Metric
- removed D2: SS24, Diode_SMD:D_SMA
- removed Q1: FDN340P, Package_TO_SOT_SMD:SOT-23
- removed U7: KA78M05, Package_TO_SOT_SMD:TO-252-2
- removed U9: LTC4412, Package_TO_SOT_SMD:TSOT-23-6
- D4: value WS2812B -> SK6812; footprint LED_SMD:LED_WS2812B_PLCC4_5.0x5.0mm_P3.2mm -> LED_SMD:LED_SK6812_PLCC4_5.0x5.0mm_P3.2mm
- moved F1 2.15 mm to (91.4, 118.2), turned to -90 degrees
- moved R9 1.75 mm to (100.1, 95.8)
- moved SW1 0.88 mm to (110.3, 124.3)
- moved SW2 0.87 mm to (114.7, 124.3)
- moved TX4 0.70 mm to (132.4, 124.8)
- moved R48 0.53 mm to (135.2, 124.8)
- moved C32 0.43 mm to (115.7, 104.1)
- moved D5 0.10 mm to (149.4, 121.1)
- turned D3 to 0 degrees
- turned D4 to -90 degrees
Connections:
- net /USB_DM renamed /USB_DN
- BZ1 pad 1: VCC -> +3.3V
- D4 pad 1: +5V -> GND
- D4 pad 2: unconnected-(D4-DOUT-Pad2) -> /LED
- D4 pad 3: GND -> +3.3V
- D4 pad 4: /LED -> unconnected-(D4-DOUT-Pad4)
Routing:
- net +3.3V: track 0.00 -> 233.8 mm, vias 0 -> 12
- net VCC: track 0.00 -> 72.8 mm, vias 0 -> 2
- net PYRO_1: track 0.00 -> 53.6 mm, vias 0 -> 2
- net PYRO_2: track 0.00 -> 51.9 mm, vias 0 -> 2
- net TIM4_CH4: track 0.00 -> 45.1 mm, vias 0 -> 2
- net LORA_MISO: track 0.00 -> 38.5 mm, vias 0 -> 3
- net BAT_VSENCE: track 0.00 -> 38.4 mm, vias 0 -> 2
- net LORA_DIO1: track 0.00 -> 36.9 mm, vias 0 -> 1
- net LORA_IO0: track 0.00 -> 36.6 mm, vias 0 -> 1
- net TIM4_CH3: track 0.00 -> 36.4 mm, vias 0 -> 2
- net GPS_SCL: track 0.00 -> 35.1 mm, vias 0 -> 1
- net GPS_SDA: track 0.00 -> 34.8 mm, vias 0 -> 1
- net Net-(U1-NRST): track 0.00 -> 34.0 mm, vias 0 -> 4
- net VBUS: track 0.00 -> 33.9 mm, vias 0 -> 4
- net LORA_MOSI: track 0.00 -> 32.0 mm, vias 0 -> 3
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- added copper zone on B.Cu, net +3.3V
- added copper zone on F.Cu, net +3.3VB
- added copper zone on F.Cu, net +BATT
- added copper zone on B.Cu, net GND
- added copper zone on F.Cu, net GND
- added copper zone on F.Cu, net Net-(BZ1--)
- added copper zone on F.Cu, net Net-(U6-SW)
- added copper zone on F.Cu, net VCC
Other:
- board size 86.8 x 49.2 mm -> 86.8 x 48.2 mm
