File: Hardware/flight_comp.kicad_pcb (KiCad board)
At the start: 4 copper layers, 86.7 x 48.2 mm, 126 parts, among them IC1 BMP388, IC4 TPS259531DSGR, J1 Conn_Coaxial, J10 CAMERA_CONN_01, J11 CAMERA_CONN_02, J12 Conn_Coaxial, J13 CAMERA_CONN_03, J2 TC2030, J3 XT30, J4 USB_C_Receptacle_USB2.0_16P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

Commit message: Kondensators
Parts:
- added C25: 1000uF, Capacitor_THT:CP_Axial_L10.0mm_D6.0mm_P15.00mm_Horizontal, B.Cu at (93.0, 115.1)
- moved D6 0.36 mm to (101.3, 120.3)
